Commit message: Update

File: urdf/gps_wamv.xacro (robot description, xacro)
@@ -7,7 +7,7 @@
 	<alwaysOn>true</alwaysOn>
         <bodyName>gps</bodyName>
-        <frameId>gps</frameId>
-	<topicName>fix</topicName>
-        <velocityTopicName>fix_velocity</velocityTopicName>
+        <frameId>rowbot/gps</frameId>
+	<topicName>rowbot/fix</topicName>
+        <velocityTopicName>rowbot/fix_velocity</velocityTopicName>
 	<!-- Location of origin of Gazebo Sand Island map -->
 	<referenceLatitude>21.30996</referenceLatitude>

File: urdf/imu_wamv.xacro (robot description, xacro)
@@ -8,6 +8,6 @@
         <updateRate>10.0</updateRate>
         <bodyName>base_link</bodyName>
-        <topicName>imu/data</topicName>
-        <serviceName>imu_service</serviceName>
+        <topicName>rowbot/imu/data</topicName>
+        <serviceName>rowbot/imu_service</serviceName>
         <frameId>base_link</frameId>
         <alwaysOn>true</alwaysOn>

File: urdf/rowbot_wamv.xacro (robot description, xacro)
@@ -29,4 +29,6 @@
   <xacro:include filename="$(find nps_robotx)/urdf/p3d_wamv.xacro" />
   <xacro:p3d_wamv name="p3d_wamv"/-->
+  <xacro:include filename="$(find rowbot_description)/urdf/magnetic_wamv.xacro" />
+  <xacro:magnetic_wamv name="magnetic_wamv"/>
   <xacro:include filename="$(find pointgrey_camera_description)/urdf/pointgrey_flea3.urdf.xacro" />
   <xacro:pointgrey_flea3 frame="mycamera"/>
@@ -37,6 +39,6 @@
   </joint>
   <xacro:include filename="$(find velodyne_description)/urdf/VLP-16.urdf.xacro"/>
-  <VLP-16 parent="base_link" name="velodyne" topic="/velodyne_points" hz="10" samples="440">
-    <origin xyz="0.8 0 1.3" rpy="0 0 0" />
+  <VLP-16 parent="base_link" name="velodyne" topic="rowbot/velodyne_points" hz="10" samples="440">
+    <origin xyz="0.8 0 1.8" rpy="0 0 0" />
   </VLP-16>
 <!--<gazebo reference="scan">
