Commit message: CHanged camera

File: urdf/front_camera_wamv.xacro (robot description, xacro)
@@ -7,8 +7,8 @@
       <update_rate>30.0</update_rate>
       <camera name="head">
-        <horizontal_fov>1.3962634</horizontal_fov>
+        <horizontal_fov>1.22173</horizontal_fov>
         <image>
-          <width>800</width>
-          <height>800</height>
+          <width>1280</width>
+          <height>720</height>
           <format>R8G8B8</format>
         </image>
@@ -29,7 +29,7 @@
         <alwaysOn>true</alwaysOn>
         <updateRate>0.0</updateRate>
-        <cameraName>wamv_camera_front</cameraName>
-        <imageTopicName>image_raw</imageTopicName>
-        <cameraInfoTopicName>camera_info</cameraInfoTopicName>
+        <!--cameraName>wamv_camera_front</cameraName-->
+        <imageTopicName>rowbot/image_raw</imageTopicName>
+        <cameraInfoTopicName>rowbot/camera_info</cameraInfoTopicName>
         <frameName>front_camera_link</frameName>
         <hackBaseline>0.07</hackBaseline>

File: urdf/gps_wamv.xacro (robot description, xacro)
@@ -7,7 +7,7 @@
 	<alwaysOn>true</alwaysOn>
         <bodyName>gps</bodyName>
-        <frameId>rowbot/gps</frameId>
-	<topicName>rowbot/fix</topicName>
-        <velocityTopicName>rowbot/fix_velocity</velocityTopicName>
+        <frameId>gps</frameId>
+	<topicName>rowbot/gps/fix</topicName>
+        <velocityTopicName>rowbot/gps/fix_velocity</velocityTopicName>
 	<!-- Location of origin of Gazebo Sand Island map -->
 	<referenceLatitude>21.30996</referenceLatitude>

File: urdf/rowbot_wamv.xacro (robot description, xacro)
@@ -14,7 +14,7 @@
   <xacro:usv_thrust_gazebo name="wamv_thrust_plugin"/>
   <!-- ADD SENSORS -->
-  <!-- Add a front camera >
+  <!-- Add a front camera -->
  <xacro:include filename="$(find rowbot_description)/urdf/front_camera_wamv.xacro" />
-  <xacro:wamv_camera name="wamv_front_camera"/-->
+  <xacro:wamv_camera name="wamv_front_camera"/>
     <!-- Add simulated Multibeam >
     <xacro:include filename="$(find nps_robotx)/urdf/multibeam_wamv.xacro" />
@@ -24,5 +24,5 @@
   <xacro:gps_wamv name="gps_wamv"/>
   <!-- Add Simulated IMU -->
-  <xacro:include filename="$(find nps_robotx)/urdf/imu_wamv.xacro" />
+  <xacro:include filename="$(find rowbot_description)/urdf/imu_wamv.xacro" />
   <xacro:imu_wamv name="imu_wamv"/>
   <!-- Add P3D ground truth -->
@@ -31,5 +31,5 @@
   <xacro:include filename="$(find rowbot_description)/urdf/magnetic_wamv.xacro" />
   <xacro:magnetic_wamv name="magnetic_wamv"/>
-  <xacro:include filename="$(find pointgrey_camera_description)/urdf/pointgrey_flea3.urdf.xacro" />
+  <!--xacro:include filename="$(find pointgrey_camera_description)/urdf/pointgrey_flea3.urdf.xacro" />
   <xacro:pointgrey_flea3 frame="mycamera"/>
   <joint name="mycamera_joint" type="fixed">
@@ -37,5 +37,5 @@
     <parent link="base_link"/>
     <child link="mycamera"/>
-  </joint>
+  </joint-->
   <xacro:include filename="$(find velodyne_description)/urdf/VLP-16.urdf.xacro"/>
   <VLP-16 parent="base_link" name="velodyne" topic="rowbot/velodyne_points" hz="10" samples="440">
