Commit message: Compatiable with new simulatoin

File: urdf/rowbot_wamv.xacro (robot description, xacro)
@@ -2,68 +2,16 @@
 <robot xmlns:xacro="http://ros.org/wiki/xacro"
        name="WAM-V">
-    <!-- Defines the base vehicle -->
-  <xacro:include filename="$(find wamv_description)/urdf/wamv_base.xacro" />
-  <!-- Attach hydrodynamics plugin -->
-  <xacro:include filename="$(find robotx_gazebo)/urdf/wamv_gazebo_dynamics_plugin.xacro" />
-  <xacro:usv_dynamics_gazebo name="wamv_dynamics_plugin"/>
-  <!-- Attach wind plugin -->
-  <xacro:include filename="$(find robotx_gazebo)/urdf/wamv_gazebo_wind_plugin.xacro" />
-  <xacro:usv_wind_gazebo name="wamv_wind_plugin"/>
-  <!-- Attach thrust plugin -->
-  <xacro:include filename="$(find robotx_gazebo)/urdf/wamv_gazebo_thrust_plugin.xacro" />
-  <xacro:usv_thrust_gazebo name="wamv_thrust_plugin"/>
-  <!-- ADD SENSORS -->
-  <!-- Add a front camera -->
- <xacro:include filename="$(find rowbot_description)/urdf/front_camera_wamv.xacro" />
-  <xacro:wamv_camera name="wamv_front_camera"/>
-    <!-- Add simulated Multibeam >
-    <xacro:include filename="$(find nps_robotx)/urdf/multibeam_wamv.xacro" />
-    <xacro:multibeam_wamv name="multibeam_wamv"/-->
-   <!-- Add simulated GPS -->
-  <xacro:include filename="$(find rowbot_description)/urdf/gps_wamv.xacro" />
-  <xacro:gps_wamv name="gps_wamv"/>
+  <!-- WAMV with "T" thruster configuration -->
+  <xacro:include filename="$(find rowbot_description)/urdf/wamv_gazebo.urdf.xacro" />
+  <!-- ==== VMRC sensor configuration ==== -->
+  <!-- Add a cameras camera pair -->
+  <xacro:wamv_camera name="left_camera" y="0.2" x="0.75" Y="${radians(60)}" />
+  <xacro:wamv_camera name="front_camera" x="0.75" z="1.35" />
+  <xacro:wamv_camera name="right_camera" y="-0.2" x="0.75" Y="${radians(-60)}" />
+  <!-- Add simulated GPS -->
+  <xacro:wamv_gps name="gps_wamv" y="0.2" />
   <!-- Add Simulated IMU -->
-  <xacro:include filename="$(find rowbot_description)/urdf/imu_wamv.xacro" />
-  <xacro:imu_wamv name="imu_wamv"/>
-  <!-- Add P3D ground truth -->
-  <xacro:include filename="$(find rowbot_description)/urdf/p3d_wamv.xacro" />
-  <xacro:p3d_wamv name="p3d_wamv"/>
-  <xacro:include filename="$(find rowbot_description)/urdf/magnetic_wamv.xacro" />
-  <xacro:magnetic_wamv name="magnetic_wamv"/>
-  <!--xacro:include filename="$(find pointgrey_camera_description)/urdf/pointgrey_flea3.urdf.xacro" />
-  <xacro:pointgrey_flea3 frame="mycamera"/>
-  <joint name="mycamera_joint" type="fixed">
-    <origin xyz="0.5 0 1.5"/>
-    <parent link="base_link"/>
-    <child link="mycamera"/>
-  </joint-->
-  <xacro:include filename="$(find velodyne_description)/urdf/VLP-16.urdf.xacro"/>
-  <VLP-16 parent="base_link" name="velodyne" topic="rowbot/velodyne_points" hz="10" samples="440">
-    <origin xyz="0.8 0 1.8" rpy="0 0 0" />
-  </VLP-16>
-<!--<gazebo reference="scan">
-    <sensor type="gpu_ray" name="multibeam">
-        <visualize>true</visualize>
-        <update_rate>10</update_rate>
-        <ray>
-            <scan>
-                <horizontal>
-                    <samples>256</samples>
-                    <resolution>1</resolution>
-                    <min_angle>-1.0472</min_angle>
-                    <max_angle>1.0472</max_angle>
-                </horizontal>
-            </scan>
-            <range>
-                <min>0.2</min>
-                <max>70</max>
-                <resolution>0.02</resolution>
-            </range>
-        </ray>
-        <plugin name="gazebo_ros_head_hokuyo_controller" filename="libgazebo_ros_gpu_laser.so">
-            <topicName>/kayak/multibeam/scan</topicName>
-            <frameName>scan</frameName>
-        </plugin>
-    </sensor>
-</gazebo>-->
+  <xacro:wamv_imu name="imu_wamv" y="-0.2" />
+  <!-- Add 3D LIDAR -->
+  <xacro:wamv_3d_lidar name="lidar_wamv" />
 </robot>
